File: Diamond.kicad_sch (KiCad schematic)
At the start: 0 parts

Commit message: Added Sheets
Other:
- note added: "Diamond"
Changed lines of the file:
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@@
 	(generator_version "10.0")
 	(paper "A4")
+	(text "Diamond"
+		(exclude_from_sim no)
+		(at 140.97 27.432 0)
+		(effects
+			(font
+				(size 12.7 12.7)
+			)
+		)
+	)
 	(sheet_instances
 		(path "/"
-			(page "3")
+			(page "1")
 		)
 	)
+	(embedded_fonts no)
 )
