File: Diamond.kicad_pcb (KiCad board)
At the start: 2 copper layers, 40 parts, among them J1 SWD, J3 USB_C_Receptacle_USB2.0_16P, Q1 SSD2300, Q2 SSD2300, Q3 SSD2300, Q4 SSD2300, U1 AP63205WU, U2 AP2112K-3.3, U3 STM32H503CBUx, U4 TPS2116DRL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

Commit message: Started PCB
Parts:
- added C14: 100n, Capacitor_SMD:C_0402_1005Metric, F.Cu at (131.0, 75.5)
- added C15: 1u, Capacitor_SMD:C_0603_1608Metric, F.Cu at (127.5, 75.8)
- added C16: 1u, Capacitor_SMD:C_0603_1608Metric, F.Cu at (127.5, 78.3)
- added C17: 100n, Capacitor_SMD:C_0402_1005Metric, F.Cu at (131.0, 77.5)
- added C18: 22u, Capacitor_SMD:C_0805_2012Metric, F.Cu at (121.3, 98.6)
- added C19: 1u, Capacitor_SMD:C_0603_1608Metric, F.Cu at (121.1, 75.8)
- added C20: 1u, Capacitor_SMD:C_0603_1608Metric, F.Cu at (121.1, 78.3)
- added C21: 1u, Capacitor_SMD:C_0603_1608Metric, F.Cu at (121.1, 80.8)
- added C22: 100n, Capacitor_SMD:C_0402_1005Metric, F.Cu at (120.5, 101.1)
- added C23: 100n, Capacitor_SMD:C_0402_1005Metric, F.Cu at (120.5, 103.1)
- added J4: Conn_01x21_Pin, Connector_PinSocket_2.54mm:PinSocket_1x21_P2.54mm_Vertical, F.Cu at (123.9, 131.6)
- added R14: 5k1, Resistor_SMD:R_0603_1608Metric, F.Cu at (127.5, 80.8)
- added R15: 10k, Resistor_SMD:R_0603_1608Metric, F.Cu at (127.5, 83.3)
- added R16: 27, Resistor_SMD:R_0603_1608Metric, F.Cu at (127.5, 85.8)
- added R17: 27, Resistor_SMD:R_0603_1608Metric, F.Cu at (127.5, 88.3)
- added R18: 4k7, Resistor_SMD:R_0603_1608Metric, F.Cu at (121.1, 83.3)
- added R19: 4k7, Resistor_SMD:R_0603_1608Metric, F.Cu at (121.1, 85.8)
- added R20: 4k7, Resistor_SMD:R_0603_1608Metric, F.Cu at (121.1, 88.3)
- added R21: 4k7, Resistor_SMD:R_0603_1608Metric, F.Cu at (121.1, 90.8)
- added R22: 4k7, Resistor_SMD:R_0603_1608Metric, F.Cu at (121.1, 93.3)
- added R23: 4k7, Resistor_SMD:R_0603_1608Metric, F.Cu at (121.1, 95.8)
- moved J3 53.2 mm to (191.3, 80.0), turned to 90 degrees
- moved R12 38.0 mm to (172.2, 82.7)
- moved R13 38.0 mm to (172.2, 85.2)
- moved U5 38.0 mm to (167.1, 84.6)
- moved U6 38.0 mm to (176.1, 83.6)
- moved C12 24.6 mm to (179.1, 113.0)
- moved C13 24.6 mm to (179.1, 115.6)
- moved J1 24.6 mm to (179.4, 101.9)
- moved U7 24.6 mm to (186.1, 111.2)
- moved U3 16.8 mm to (145.4, 100.4)
Connections:
- net /Schematic/Power/5V_USB renamed /Schematic/USB C/VBUS
- U3 pad 10: unconnected-(U3-PA0-Pad10) -> /Schematic/MCU/MISO
- U3 pad 11: unconnected-(U3-PA1-Pad11) -> /Schematic/MCU/CS
- U3 pad 12: unconnected-(U3-PA2-Pad12) -> /Schematic/MCU/SCLK
- U3 pad 14: unconnected-(U3-PA4-Pad14) -> /Schematic/MCU/MOSI
- U3 pad 25: unconnected-(U3-PB12-Pad25) -> /Schematic/MCU/CANRX
- U3 pad 26: unconnected-(U3-PB13-Pad26) -> /Schematic/MCU/CANTX
- U3 pad 32: unconnected-(U3-PA11-Pad32) -> /Schematic/MCU/DM
- U3 pad 33: unconnected-(U3-PA12-Pad33) -> /Schematic/MCU/DP
- U3 pad 34: unconnected-(U3-PA13(JTMS-Pad34) -> /Schematic/MCU/SWDIO
- U3 pad 37: unconnected-(U3-PA14(JTCK-Pad37) -> /Schematic/MCU/SWCLK
- U3 pad 38: unconnected-(U3-PA15(JTDI)-Pad38) -> /Schematic/MCU/SWO
- U3 pad 44: unconnected-(U3-BOOT0-Pad44) -> /Schematic/MCU/BOOT0
- U3 pad 7: unconnected-(U3-NRST-Pad7) -> /Schematic/MCU/RST
- U5 pad 4: unconnected-(U5-CBUS4-Pad4) -> Net-(U5-CBUS4)
- U5 pad 6: /Schematic/USB C/DP_2 -> Net-(U5-USBDP)
- U5 pad 7: /Schematic/USB C/DM_2 -> Net-(U5-USBDM)
- U7 pad 1: unconnected-(U7-VCAP-Pad1) -> Net-(U7-VCAP)
- U7 pad 2: unconnected-(U7-A1-Pad2) -> GND
- U7 pad 3: unconnected-(U7-A2-Pad3) -> GND
- U7 pad 4: unconnected-(U7-VSS-Pad4) -> GND
- U7 pad 5: unconnected-(U7-SDA-Pad5) -> /Schematic/MCU/SDA
- U7 pad 6: unconnected-(U7-SCL-Pad6) -> /Schematic/MCU/SCL
- U7 pad 7: unconnected-(U7-HS-Pad7) -> GND
- U7 pad 8: unconnected-(U7-VCC-Pad8) -> +3V3
Other:
- board outline added: 95 x 70 mm
- copper layers 2 -> 4
